File: Rudie's Bass Fuzz.kicad_pcb (KiCad board)
At the start: 2 copper layers, 25 x 50 mm, 19 parts, among them J1 Conn_01x01_Male, J2 Conn_01x01_Male, J3 Conn_01x01_Male, J4 Conn_01x01_Male, J5 Conn_01x01_Male, J6 Conn_01x01_Male, Q1 BC549

Commit message: corrected spelling mistake
bazz fuzz -> bazz fuss (joke)
Other:
- board text added: "Rudie's gore Bazz Fuss"
- board text added: "Rudie's gore Bazz Fuss V0.1 15-12-2022"
- board text removed: "Rudie's gore Bazz Fuzz"
- board text removed: "Rudie's gore Bazz Fuzz V0.1 15-12-2022"
Changed lines of the file:
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@@
   (gr_arc (start 183.6 92) (mid 183.424264 92.424264) (end 183 92.6) (layer "Edge.Cuts") (width 0.1))
   (gr_arc (start 183 42.6) (mid 183.424264 42.775736) (end 183.6 43.2) (layer "Edge.Cuts") (width 0.1))
-  (gr_text "Rudie's gore \nBazz Fuzz V0.1\n15-12-2022" (at 177.927 76.835 90) (layer "B.SilkS")
+  (gr_text "Rudie's gore \nBazz Fuss V0.1\n15-12-2022" (at 177.927 76.835 90) (layer "B.SilkS")
     (effects (font (size 1 1) (thickness 0.15)) (justify left mirror))
   )
@@
     (effects (font (size 1 1) (thickness 0.15)))
   )
-  (gr_text "Rudie's gore \nBazz Fuzz" (at 175.768 67.564 90) (layer "F.SilkS")
+  (gr_text "Rudie's gore \nBazz Fuss" (at 175.768 67.564 90) (layer "F.SilkS")
     (effects (font (size 1.2 1.2) (thickness 0.17)))
   )
